Commit message: rviz, pgm (no map though), and teleop

File: catkin_ws/src/my_robot/urdf/my_robot.xacro (robot description, xacro)
@@ -131,5 +131,5 @@
       />
     </inertial>
-    <collision name='collision'>
+    <collision name='camera_collision'>
       <origin xyz="0 0 0" rpy=" 0 0 0"/>
       <geometry>
@@ -163,5 +163,5 @@
       />
     </inertial>
-    <collision name='collision'>
+    <collision name='hokuyo_collision'>
       <origin xyz="0 0 0" rpy=" 0 0 0"/>
       <geometry>

Commit message: newest changes

File: catkin_ws/src/my_robot/urdf/my_robot.xacro (robot description, xacro)
@@ -131,5 +131,5 @@
       />
     </inertial>
-    <collision name='camera_collision'>
+    <collision name='collision'>
       <origin xyz="0 0 0" rpy=" 0 0 0"/>
       <geometry>
@@ -163,5 +163,5 @@
       />
     </inertial>
-    <collision name='hokuyo_collision'>
+    <collision name='collision'>
       <origin xyz="0 0 0" rpy=" 0 0 0"/>
       <geometry>
